File: _autosave-macropad.kicad_pcb (KiCad board)
At the start: 2 copper layers, 87.5 x 56 mm, 17 parts, among them J1 Oled Pins, SW2 SW_Push, SW3 SW_Push, SW4 SW_Push, SW5 SW_Push, SW6 SW_Push, SW7 SW_Push, U1 Seeed Studio XIAO SAMD21

Commit message: Finished pcb
Parts:
- moved J1 1.50 mm to (143.5, 76.0)
Routing:
- net VCC: track 101.7 -> 103.6 mm
- net GND: track 109.9 -> 111.2 mm
- net SCL: track 57.5 -> 56.9 mm
- net SDA: track 58.8 -> 58.1 mm
Changed lines of the file:
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@@
 	(footprint "Connector_PinHeader_1.00mm:PinHeader_1x04_P1.00mm_Vertical"
 		(layer "F.Cu")
-		(at 143.5 74.5)
+		(at 143.5 76)
 		(descr "Through hole straight pin header, 1x04, 1.00mm pitch, single row")
 		(tags "Through hole pin header THT 1x04 1.00mm single row")
@@
 	)
 	(gr_rect
-		(start 142 69.5)
-		(end 182 82.5)
+		(start 142 71)
+		(end 182 84)
 		(stroke
 			(width 0.1)
@@
 	)
 	(segment
-		(start 143.5 77.5)
-		(end 144.10104 77.5)
-		(width 0.2)
-		(layer "F.Cu")
-		(net 1)
-	)
-	(segment
 		(start 111 115.7)
 		(end 110.25 116.45)
@@
 	)
 	(segment
+		(start 143.666726 79)
+		(end 143.5 79)
+		(width 0.2)
+		(layer "F.Cu")
+		(net 1)
+	)
+	(segment
 		(start 112.66 70.71)
 		(end 115.6 73.65)
@@
 	)
 	(segment
+		(start 144.625 78.041726)
+		(end 143.666726 79)
+		(width 0.2)
+		(layer "F.Cu")
+		(net 1)
+	)
+	(segment
 		(start 144.625 73.609314)
 		(end 142.125686 71.11)
@@
 	)
 	(segment
-		(start 144.10104 77.5)
-		(end 144.625 76.97604)
-		(width 0.2)
-		(layer "F.Cu")
-		(net 1)
-	)
-	(segment
-		(start 144.625 76.97604)
-		(end 144.625 73.609314)
+		(start 144.625 73.609314)
+		(end 144.625 78.041726)
 		(width 0.2)
 		(layer "F.Cu")
@@
 	)
 	(segment
+		(start 144.10104 78)
+		(end 143.5 78)
+		(width 0.2)
+		(layer "F.Cu")
+		(net 12)
+	)
+	(segment
 		(start 117.226346 75.95)
 		(end 117.9 75.276346)
@@
 	)
 	(segment
-		(start 144.225 75.800305)
-		(end 144.225 73.775)
+		(start 144.225 73.775)
+		(end 144.225 77.87604)
 		(width 0.2)
 		(layer "F.Cu")
@@
 	)
 	(segment
-		(start 143.5 76.5)
-		(end 143.525305 76.5)
-		(width 0.2)
-		(layer "F.Cu")
-		(net 12)
-	)
-	(segment
-		(start 143.525305 76.5)
-		(end 144.225 75.800305)
+		(start 144.225 77.87604)
+		(end 144.10104 78)
 		(width 0.2)
 		(layer "F.Cu")
@@
 	)
 	(segment
+		(start 141.375 76)
+		(end 143.5 76)
+		(width 0.2)
+		(layer "F.Cu")
+		(net 15)
+	)
+	(segment
 		(start 138.52 78.855)
 		(end 138.52 89.999899)
@@
 	)
 	(segment
-		(start 142.875 74.5)
-		(end 138.52 78.855)
-		(width 0.2)
-		(layer "F.Cu")
-		(net 15)
-	)
-	(segment
-		(start 143.5 74.5)
-		(end 142.875 74.5)
-		(width 0.2)
-		(layer "F.Cu")
-		(net 15)
-	)
-	(segment
 		(start 136.540101 90.82)
 		(end 135.72 89.999899)
@@
 	)
 	(segment
+		(start 138.52 78.855)
+		(end 141.375 76)
+		(width 0.2)
+		(layer "F.Cu")
+		(net 15)
+	)
+	(segment
 		(start 135.72 89.999899)
 		(end 109.079899 89.999899)
@@
 	)
 	(segment
-		(start 142.89896 75.5)
-		(end 139.042793 79.356167)
-		(width 0.2)
-		(layer "F.Cu")
-		(net 16)
-	)
-	(segment
-		(start 143.5 75.5)
-		(end 142.89896 75.5)
+		(start 139.042793 79.356167)
+		(end 141.39896 77)
 		(width 0.2)
 		(layer "F.Cu")
@@
 		(width 0.2)
 		(layer "F.Cu")
+		(net 16)
+	)
+	(segment
+		(start 141.39896 77)
+		(end 143.5 77)
+		(width 0.2)
+		(layer "F.Cu")
